File: Inverter V3.brd (EAGLE design)
At the start: 262.4 x 114 mm, 67 parts, among them IC1 LTV-816, IC2 LTV-816, IC3 LTV-816, IC4 LTV-816, IC5 LTV-816, IC6 LTV-816, Q1 ROHM_SCT3022ALGC11ROHM_SCT302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, Q2 ROHM_SCT3022ALGC11ROHM_SCT302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, Q3 ROHM_SCT3022ALGC11ROHM_SCT302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, Q4 ROHM_SCT3022ALGC11ROHM_SCT302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, Q5 ROHM_SCT3022ALGC11ROHM_SCT302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, Q6 ROHM_SCT3022ALGC11ROHM_SCT302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, U1 RASPBERRY_PICOTH

Commit message: Swapped flyback diodes and added silkscreen for IC pins
Parts:
- removed D4, D5, D6, D7, D8, D9: 1N4004, diode:DO41-10
- added D16, D17, D18, D19, D20, D21: TP1.5KE30A, TP1.5KE30A:DIOAD2855W107L835D505
- moved D14 32.1 mm to (108.8, 27.9)
- moved R16 9.02 mm to (77.5, 51.5)
- moved R15 6.92 mm to (119.2, 69.6)
- moved D12 6.66 mm to (77.5, 47.5)
- moved R9 5.25 mm to (87.1, 66.8)
- moved R12 0.87 mm to (146.1, 45.1)
- moved D11 0.80 mm to (104.8, 67.4)
- moved R7 0.20 mm to (153.5, 78.2)
Connections:
- net LO2: now also D19.1; no longer D5.C
- net SHUNT: now also D19.2, D20.2, D21.2; no longer D5.A, D7.A, D9.A
- net V+: now also D16.1, D17.1, D18.1; no longer D4.C, D6.C, D8.C
- net VOUT3/VS3: now also D18.2, D21.1; no longer D8.A, D9.C
- net VS1/VOUT1: now also D16.2; no longer D4.A
- net VS2/VOUT2: now also D17.2, D20.1; no longer D6.A, D7.C
Routing:
- net LO2: track 87.9 -> 142.3 mm, vias 3 -> 2
- net VGIN5: track 94.6 -> 129.6 mm, vias 1 -> 2
- net VGIN3: track 149.2 -> 127.7 mm, vias 2 -> 4
- net SHUNT: track 322.1 -> 343.4 mm, vias 1 -> 0
- net VOUT3/VS3: track 263.0 -> 284.0 mm, vias 3 -> 2
- net V+: track 161.6 -> 176.7 mm, vias 1 -> 0
- net VGIN6: track 192.9 -> 201.2 mm
- net VS2/VOUT2: track 200.8 -> 197.4 mm
- net VGIN2: track 80.2 -> 83.5 mm
- net HO2: track 66.9 -> 64.5 mm
- net VS1/VOUT1: track 191.7 -> 190.0 mm, vias 1 -> 2
- net VGIN1: track 65.1 -> 64.0 mm
Other:
- board size 262.4 x 114 mm -> 248.6 x 114.2 mm
- board text added: "OC_HIN1 OC_LIN1 OC_HIN2 OC_LIN2 OC_HIN3 OC_LIN3 LO3 VOUT3 HO3 VB3"
- board text added: "VB1 HO1 VS1/VOUT1 LO1 VB2 HO2 VOUT2 LO2 VDD GND"
- board text removed: "C:/Users/leapa/Desktop/hx logo.bmp"
